Commit message: feat(lekiwi): 更新机器人硬件配置和控制参数
- 重构控制器配置文件，优化硬件参数设置
- 更新URDF模型，添加视觉材质和正确的关节连接
- 改进基类启动逻辑，增加电机使能功能
- 优化launch文件结构，简化节点启动流程
- 修复序列通信相关的问题，改进速度控制实现
```

File: src/lekiwi/urdf/lekiwi_base.urdf (robot description, URDF)
Before this commit: robot lekiwi, 4 links, 3 joints
Links:
- removed link rear_wheel_link
- removed link right_wheel_link
- link base_link: geometry visual box size=0.2 0.2 0.1
- link left_wheel_link: geometry visual cylinder length=0.02 radius=0.03
Joints:
- joint left_wheel_drive: origin (none) -> xyz=0.1 0.1 0 rpy=-1.5708 0 0
- joint rear_wheel_drive: child rear_wheel_link -> left_wheel_link; origin (none) -> xyz=0 -0.1 0 rpy=-1.5708 0 0
- joint right_wheel_drive: child right_wheel_link -> left_wheel_link; origin (none) -> xyz=-0.1 0.1 0 rpy=-1.5708 0 0
